Commit message: Tiny Pushes

File: description/robot_core.xacro (robot description, xacro)
@@ -20,4 +20,10 @@
     <link name="base_link" >
     </link>
+    <!-- BASE FOOTPRINT LINK -->
+    <joint name="base_footprint_joint" type="fixed">
+        <parent link="base_link" />
+        <child link="base_footprint" />
+        <origin xyz="0 0 0" rpy="0 0 0"/>
+    </joint>
     <!-- CHASSIS LINK -->
     <joint name="chassis_joint" type="fixed">
