Commit message: Added YDLidar launch file

File: description/lidar.xacro (robot description, xacro)
@@ -1,3 +1,14 @@
 <?xml version="1.0"?>
+<robot xmlns:xacro="http://www.ros.org/wiki/xacro" >
+    <joint name="laser_joint" type="fixed">
+        <parent link="chassis"/>
+        <child link="laser_frame"/>
+        <origin xyz="0.27 0 0.1075" rpy="0 0 0"/>
+    </joint>
+    <link name="laser_frame">
+    <visual>
+            <geometry>
+                <cylinder radius="0.03" length="0.02"/>
+            </geometry><?xml version="1.0"?>
 <robot xmlns:xacro="http://www.ros.org/wiki/xacro" >
     <joint name="laser_joint" type="fixed">
@@ -48,2 +59,39 @@
     </gazebo>
 </robot>
+            <material name="red"/>
+        </visual>
+        <collision>
+            <geometry>
+                <cylinder radius="0.03" length="0.015"/>
+            </geometry>
+        </collision>
+        <xacro:inertial_cylinder mass="0.1" radius="0.03" length="0.015">
+            <origin xyz="0 0 0" rpy="0 0 0"/>
+        </xacro:inertial_cylinder>
+    </link>
+    <gazebo reference="laser_frame">
+        <material>Gazebo/Red</material>
+        <sensor name="laser" type="gpu_lidar">
+            <pose> 0 0 0 0 0 0 </pose>
+            <visualize>true</visualize>
+            <update_rate>10</update_rate>
+            <lidar>
+                <scan>
+                    <horizontal>
+                        <samples>360</samples>
+                        <resolution>1</resolution>
+                        <min_angle>-3.14</min_angle>
+                        <max_angle>3.14</max_angle>
+                    </horizontal>
+                </scan>
+                <range>
+                    <min>0.6</min>
+                    <max>8</max>
+                    <resolution>0.01</resolution>
+                </range>
+            </lidar>
+            <topic>scan</topic>
+            <gz_frame_id>laser_frame</gz_frame_id>
+        </sensor>
+    </gazebo>
+</robot>

File: description/ros2_control.xacro (robot description, xacro)
@@ -8,5 +8,5 @@
                 <param name="right_wheel_name">right_wheel_joint</param>
                 <param name="loop_rate">30</param>
-                <param name="device">/dev/ttyUSB0</param>
+                <param name="device">/dev/ttyACM0</param>
                 <param name="baud_rate">57600</param>
                 <param name="timeout">1000</param>

Commit message: Fixed to Robot Launch File

File: description/lidar.xacro (robot description, xacro)
@@ -7,16 +7,5 @@
     </joint>
     <link name="laser_frame">
-    <visual>
-            <geometry>
-                <cylinder radius="0.03" length="0.02"/>
-            </geometry><?xml version="1.0"?>
-<robot xmlns:xacro="http://www.ros.org/wiki/xacro" >
-    <joint name="laser_joint" type="fixed">
-        <parent link="chassis"/>
-        <child link="laser_frame"/>
-        <origin xyz="0.27 0 0.1075" rpy="0 0 0"/>
-    </joint>
-    <link name="laser_frame">
-    <visual>
+        <visual>
             <geometry>
                 <cylinder radius="0.03" length="0.02"/>
@@ -59,39 +48,2 @@
     </gazebo>
 </robot>
-            <material name="red"/>
-        </visual>
-        <collision>
-            <geometry>
-                <cylinder radius="0.03" length="0.015"/>
-            </geometry>
-        </collision>
-        <xacro:inertial_cylinder mass="0.1" radius="0.03" length="0.015">
-            <origin xyz="0 0 0" rpy="0 0 0"/>
-        </xacro:inertial_cylinder>
-    </link>
-    <gazebo reference="laser_frame">
-        <material>Gazebo/Red</material>
-        <sensor name="laser" type="gpu_lidar">
-            <pose> 0 0 0 0 0 0 </pose>
-            <visualize>true</visualize>
-            <update_rate>10</update_rate>
-            <lidar>
-                <scan>
-                    <horizontal>
-                        <samples>360</samples>
-                        <resolution>1</resolution>
-                        <min_angle>-3.14</min_angle>
-                        <max_angle>3.14</max_angle>
-                    </horizontal>
-                </scan>
-                <range>
-                    <min>0.6</min>
-                    <max>8</max>
-                    <resolution>0.01</resolution>
-                </range>
-            </lidar>
-            <topic>scan</topic>
-            <gz_frame_id>laser_frame</gz_frame_id>
-        </sensor>
-    </gazebo>
-</robot>

File: description/robot_core.xacro (robot description, xacro)
@@ -44,8 +44,8 @@
         <origin xyz="0.275 0 0.00625"/>
             <geometry>
-                <box size="0.5 0.5 0.2"/>
-            </geometry>
-        </collision>
-        <xacro:inertial_box mass="0.5" x="0.5" y="0.5" z="0.2">
+                <box size="0.16 0.16 0.0125"/>
+            </geometry>
+        </collision>
+        <xacro:inertial_box mass="0.5" x="0.55" y="0.56" z="0.0125">
             <origin xyz="0.275 0 0.00625" rpy="0 0 0"/>
         </xacro:inertial_box>
@@ -174,5 +174,4 @@
         </visual>
         <collision>
-        <origin xyz="0.27 0 0.06"/>
             <geometry>
                 <box size="0.19 0.19 0.095"/>
@@ -200,7 +199,6 @@
         </visual>
         <collision>
-        <origin xyz="0.525 -0.255 0.2125"/>
-            <geometry>
-                <box size="0.5 0.5 0.4"/>
+            <geometry>
+                <box size="0.05 0.05 0.4"/>
             </geometry>
         </collision>
@@ -226,5 +224,4 @@
         </visual>
         <collision>
-        <origin xyz="0.525 0.255 0.2125"/>
             <geometry>
                 <box size="0.05 0.05 0.4"/>
@@ -252,5 +249,4 @@
         </visual>
         <collision>
-        <origin xyz="0.025 -0.255 0.2125"/>
             <geometry>
                 <box size="0.05 0.05 0.4"/>
@@ -278,5 +274,4 @@
         </visual>
         <collision>
-        <origin xyz="0.025 0.255 0.2125"/>
             <geometry>
                 <box size="0.05 0.05 0.4"/>
@@ -304,5 +299,4 @@
         </visual>
         <collision>
-        <origin xyz="0.275 0 0.43125"/>
             <geometry>
                 <box size="0.55 0.56 0.05"/>
