Commit message: Finished Model without LiDAR

File: description/robot.urdf.xacro (robot description, xacro)
@@ -2,3 +2,4 @@
 <robot xmlns:xacro="http://www.ros.org/wiki/xacro"  name="robot">
     <xacro:include filename="robot_core.xacro" />
+    <xacro:include filename="gazebo_control.xacro" />
 </robot>

File: description/robot_core.xacro (robot description, xacro)
@@ -21,29 +21,32 @@
         <parent link="base_link"/>
         <child link="chassis"/>
-        <origin xyz="-0.1 0 0"/>
+        <origin xyz="-0.275 0 0"/>
     </joint>
     <link name="chassis">
         <visual>
-        <origin xyz="0.1 0 0.1"/>
+        <origin xyz="0.275 0 0.00625"/>
+            <geometry>
+                <box size="0.55 0.56 0.0125"/>
+            </geometry>
+            <material name="white" />
+        </visual>
+        <collision>
+        <origin xyz="0.275 0 0.00625"/>
             <geometry>
                 <box size="0.5 0.5 0.2"/>
             </geometry>
-            <material name="white" />
-        </visual>
-        <collision>
-        <origin xyz="0.1 0 0.1"/>
-            <geometry>
-                <box size="0.5 0.5 0.2"/>
-            </geometry>
         </collision>
         <xacro:inertial_box mass="0.5" x="0.5" y="0.5" z="0.2">
-            <origin xyz="0.1 0 0.1" rpy="0 0 0"/>
-        </xacro:inertial_box>
-    </link>
+            <origin xyz="0.275 0 0.00625" rpy="0 0 0"/>
+        </xacro:inertial_box>
+    </link>
+    <gazebo reference="chassis">
+        <material>Gazebo/Orange</material>
+    </gazebo>
     <!-- LEFT WHEEL LINK-->
     <joint name="left_wheel_joint" type="continuous">
         <parent link="base_link"/>
         <child link="left_wheel"/>
-        <origin xyz="0 0.15 0" rpy="-${pi/2} 0 0"/>
+        <origin xyz="0 0.17 -0.02375" rpy="-${pi/2} 0 0"/>
         <axis xyz="0 0 1"/>
     </joint>
@@ -51,5 +54,5 @@
         <visual>
             <geometry>
-                <cylinder radius="0.06" length="0.04"/>
+                <cylinder radius="0.0525" length="0.055"/>
             </geometry>
             <material name="blue"/>
@@ -57,16 +60,19 @@
         <collision>
             <geometry>
-                <cylinder radius="0.06" length="0.04"/>
-            </geometry>
-        </collision>
-        <xacro:inertial_cylinder mass="0.1" length="0.04" radius="0.06">
+                <cylinder radius="0.0525" length="0.055"/>
+            </geometry>
+        </collision>
+        <xacro:inertial_cylinder mass="0.1" length="0.055" radius="0.0525">
             <origin xyz="0 0 0" rpy="0 0 0"/>
         </xacro:inertial_cylinder>
     </link>
+    <gazebo reference="left_wheel">
+        <material>Gazebo/Blue</material>
+    </gazebo>
     <!-- RIGHT WHEEL LINK-->
     <joint name="right_wheel_joint" type="continuous">
         <parent link="base_link"/>
         <child link="right_wheel"/>
-        <origin xyz="0 -0.15 0" rpy="${pi/2} 0 0"/>
+        <origin xyz="0 -0.17 -0.02375" rpy="${pi/2} 0 0"/>
         <axis xyz="0 0 -1"/>
     </joint>
@@ -74,5 +80,5 @@
         <visual>
             <geometry>
-                <cylinder radius="0.06" length="0.04"/>
+                <cylinder radius="0.0525" length="0.055"/>
             </geometry>
             <material name="blue"/>
@@ -80,21 +86,24 @@
         <collision>
             <geometry>
-                <cylinder radius="0.06" length="0.04"/>
-            </geometry>
-        </collision>
-        <xacro:inertial_cylinder mass="0.1" length="0.04" radius="0.06">
+                <cylinder radius="0.0525" length="0.055"/>
+            </geometry>
+        </collision>
+        <xacro:inertial_cylinder mass="0.1" radius="0.0525" length="0.055">
             <origin xyz="0 0 0" rpy="0 0 0"/>
         </xacro:inertial_cylinder>
     </link>
+    <gazebo reference="right_wheel">
+        <material>Gazebo/Blue</material>
+    </gazebo>
     <!-- CASTER WHEEL TOP-->
     <joint name="caster_wheel_top_joint" type="fixed">
         <parent link="chassis"/>
         <child link="caster_wheel_top"/>
-        <origin xyz="0.25 0 0"/>
+        <origin xyz="0.44 0 -0.02375"/>
     </joint>
     <link name="caster_wheel_top">
         <visual>
             <geometry>
-                <sphere radius="0.05"/>
+                <sphere radius="0.0525"/>
             </geometry>
             <material name="black"/>
@@ -102,21 +111,26 @@
         <collision>
             <geometry>
-                <sphere radius="0.05"/>
-            </geometry>
-        </collision>
-        <xacro:inertial_sphere mass="0.1" radius="0.05">
+                <sphere radius="0.0525"/>
+            </geometry>
+        </collision>
+        <xacro:inertial_sphere mass="0.1" radius="0.0525">
             <origin xyz="0 0 0" rpy="0 0 0"/>
         </xacro:inertial_sphere>
     </link>
+    <gazebo reference="caster_wheel_top">
+        <material>Gazebo/White</material>
+        <mu1 value="0.001"/>
+        <mu2 value="0.001"/>
+    </gazebo>
         <!-- CASTER WHEEL BOTTOM-->
     <joint name="caster_wheel_bottom_joint" type="fixed">
         <parent link="chassis"/>
         <child link="caster_wheel_bottom"/>
-        <origin xyz="-0.0625 0 0"/>
+        <origin xyz="0.105 0 -0.02375"/>
     </joint>
     <link name="caster_wheel_bottom">
         <visual>
             <geometry>
-                <sphere radius="0.05"/>
+                <sphere radius="0.0525"/>
             </geometry>
             <material name="black"/>
@@ -124,10 +138,171 @@
         <collision>
             <geometry>
-                <sphere radius="0.05"/>
-            </geometry>
-        </collision>
-        <xacro:inertial_sphere mass="0.1" radius="0.05">
+                <sphere radius="0.0525"/>
+            </geometry>
+        </collision>
+        <xacro:inertial_sphere mass="0.1" radius="0.0525">
             <origin xyz="0 0 0" rpy="0 0 0"/>
         </xacro:inertial_sphere>
     </link>
+    <gazebo reference="caster_wheel_bottom">
+        <material>Gazebo/White</material>
+        <mu1 value="0.001"/>
+        <mu2 value="0.001"/>
+    </gazebo>
+        <!--   PROJECT BOX -->
+    <joint name="project_box_joint" type="fixed">
+        <parent link="chassis"/>
+        <child link="project_box"/>
+        <origin xyz="0.27 0 0.06"/>
+    </joint>
+    <link name="project_box">
+        <visual>
+            <geometry>
+                <box size="0.19 0.19 0.095"/>
+            </geometry>
+            <material name="white"/>
+        </visual>
+        <collision>
+        <origin xyz="0.27 0 0.06"/>
+            <geometry>
+                <box size="0.19 0.19 0.095"/>
+            </geometry>
+        </collision>
+        <xacro:inertial_box mass="0.5" x="0.19" y="0.19" z="0.095">
+            <origin xyz="0 0 0" rpy="0 0 0"/>
+        </xacro:inertial_box>
+    </link>
+    <gazebo reference="project_box">
+        <material>Gazebo/Orange</material>
+    </gazebo>
+            <!--   LEG 1 -->
+    <joint name="leg1_joint" type="fixed">
+        <parent link="chassis"/>
+        <child link="leg1"/>
+        <origin xyz="0.525 -0.255 0.2125"/>
+    </joint>
+    <link name="leg1">
+        <visual>
+            <geometry>
+                <box size="0.05 0.05 0.4"/>
+            </geometry>
+            <material name="white"/>
+        </visual>
+        <collision>
+        <origin xyz="0.525 -0.255 0.2125"/>
+            <geometry>
+                <box size="0.5 0.5 0.4"/>
+            </geometry>
+        </collision>
+        <xacro:inertial_box mass="0.5" x="0.05" y="0.05" z="0.4">
+            <origin xyz="0 0 0" rpy="0 0 0"/>
+        </xacro:inertial_box>
+    </link>
+    <gazebo reference="leg1">
+        <material>Gazebo/Orange</material>
+    </gazebo>
+                 <!--   LEG 2 -->
+    <joint name="leg2_joint" type="fixed">
+        <parent link="chassis"/>
+        <child link="leg2"/>
+        <origin xyz="0.525 0.255 0.2125"/>
+    </joint>
+    <link name="leg2">
+        <visual>
+            <geometry>
+                <box size="0.05 0.05 0.4"/>
+            </geometry>
+            <material name="white"/>
+        </visual>
+        <collision>
+        <origin xyz="0.525 0.255 0.2125"/>
+            <geometry>
+                <box size="0.05 0.05 0.4"/>
+            </geometry>
+        </collision>
+        <xacro:inertial_box mass="0.5" x="0.05" y="0.05" z="0.4">
+            <origin xyz="0 0 0" rpy="0 0 0"/>
+        </xacro:inertial_box>
+    </link>
+    <gazebo reference="leg2">
+        <material>Gazebo/Orange</material>
+    </gazebo>
+             <!--   LEG 3 -->
+    <joint name="leg3_joint" type="fixed">
+        <parent link="chassis"/>
+        <child link="leg3"/>
+        <origin xyz="0.025 -0.255 0.2125"/>
+    </joint>
+    <link name="leg3">
+        <visual>
+            <geometry>
+                <box size="0.05 0.05 0.4"/>
+            </geometry>
+            <material name="white"/>
+        </visual>
+        <collision>
+        <origin xyz="0.025 -0.255 0.2125"/>
+            <geometry>
+                <box size="0.05 0.05 0.4"/>
+            </geometry>
+        </collision>
+        <xacro:inertial_box mass="0.5" x="0.05" y="0.05" z="0.4">
+            <origin xyz="0 0 0" rpy="0 0 0"/>
+        </xacro:inertial_box>
+    </link>
+    <gazebo reference="leg3">
+        <material>Gazebo/Orange</material>
+    </gazebo>
+                 <!--   LEG 4 -->
+    <joint name="leg4_joint" type="fixed">
+        <parent link="chassis"/>
+        <child link="leg4"/>
+        <origin xyz="0.025 0.255 0.2125"/>
+    </joint>
+    <link name="leg4">
+        <visual>
+            <geometry>
+                <box size="0.05 0.05 0.4"/>
+            </geometry>
+            <material name="white"/>
+        </visual>
+        <collision>
+        <origin xyz="0.025 0.255 0.2125"/>
+            <geometry>
+                <box size="0.05 0.05 0.4"/>
+            </geometry>
+        </collision>
+        <xacro:inertial_box mass="0.5" x="0.05" y="0.05" z="0.4">
+            <origin xyz="0 0 0" rpy="0 0 0"/>
+        </xacro:inertial_box>
+    </link>
+    <gazebo reference="leg4">
+        <material>Gazebo/Orange</material>
+    </gazebo>
+                 <!--   TABLE TOP -->
+    <joint name="table_top_joint" type="fixed">
+        <parent link="chassis"/>
+        <child link="table_top"/>
+        <origin xyz="0.275 0 0.43125"/>
+    </joint>
+    <link name="table_top">
+        <visual>
+            <geometry>
+                <box size="0.55 0.56 0.05"/>
+            </geometry>
+            <material name="white"/>
+        </visual>
+        <collision>
+        <origin xyz="0.275 0 0.43125"/>
+            <geometry>
+                <box size="0.55 0.56 0.05"/>
+            </geometry>
+        </collision>
+        <xacro:inertial_box mass="0.5" x="0.55" y="0.56" z="0.05">
+            <origin xyz="0 0 0  " rpy="0 0 0"/>
+        </xacro:inertial_box>
+    </link>
+    <gazebo reference="table_top">
+        <material>Gazebo/Orange</material>
+    </gazebo>
 </robot>

Commit message: Phyical desciption changes

File: description/robot.urdf.xacro (robot description, xacro)
@@ -1,6 +1,6 @@
 <?xml version="1.0"?>
-<robot xmlns:xacro="http://www.ros.org/wiki/xacro"  name="robot">
+<robot xmlns:xacro="http://www.ros.org/wiki/xacro" name="robot">
     <xacro:arg name="use_ros2_control" default="true"/>
-        <xacro:arg name="sim_mode" default="false"/>
+    <xacro:arg name="sim_mode" default="false"/>
     <xacro:include filename="robot_core.xacro" />
     <xacro:if value="$(arg use_ros2_control)">
@@ -11,4 +11,3 @@
     </xacro:unless>
     <xacro:include filename="lidar.xacro" />
-    <xacro:include filename="ros2_control.xacro" />
 </robot>

File: description/ros2_control.xacro (robot description, xacro)
@@ -1,62 +1,32 @@
 <?xml version="1.0"?>
-<robot xmlns:xacro="http://www.ros.org/wiki/xacro" >
-    <xacro:unless value="$(arg sim_mode)">
-        <ros2_control name="RealRobot" type="system">
-            <hardware>
-                <plugin>diffdrive_arduino/DiffDriveArduino</plugin>
-                <param name="left_wheel_name">left_wheel_joint</param>
-                <param name="right_wheel_name">right_wheel_joint</param>
-                <param name="loop_rate">30</param>
-                <param name="device">/dev/ttyACM0</param>
-                <param name="baud_rate">57600</param>
-                <param name="timeout">1000</param>
-                <param name="enc_counts_per_rev">3450</param>
-            </hardware>
-            <joint name="left_wheel_joint">
-                <command_interface name="velocity">
-                    <param name="min">-10</param>
-                    <param name="max">10</param>
-                </command_interface>
-                <state_interface name="position" />
-                <state_interface name="velocity" />
-            </joint>
-            <joint name="right_wheel_joint">
-                <command_interface name="velocity">
-                    <param name="min">-10</param>
-                    <param name="max">10</param>
-                </command_interface>
-                <state_interface name="position" />
-                <state_interface name="velocity" />
-            </joint>
-        </ros2_control>
-    </xacro:unless>
-    <xacro:if value="$(arg sim_mode)">
-        <ros2_control name="GazeboSystem" type="system">
-            <hardware>
-                <plugin>gz_ros2_control/GazeboSimSystem</plugin>
-            </hardware>
-            <joint name="left_wheel_joint">
-                <command_interface name="velocity">
-                    <param name="min">-10</param>
-                    <param name="max">10</param>
-                </command_interface>
-                <state_interface name="position" />
-                <state_interface name="velocity" />
-            </joint>
-            <joint name="right_wheel_joint">
-                <command_interface name="velocity">
-                    <param name="min">-10</param>
-                    <param name="max">10</param>
-                </command_interface>
-                <state_interface name="position" />
-                <state_interface name="velocity" />
-            </joint>
-        </ros2_control>
-    </xacro:if>
-    <gazebo>
-        <plugin name="gz_ros2_control::GazeboSimROS2ControlPlugin" filename="libgz_ros2_control-system.so">
-            <parameter>$(find mobile_table)/config/my_controllers.yaml</parameter>
-            <parameter>$(find mobile_table)/config/gaz_ros2_ctl_use_sim.yaml</parameter>
-        </plugin>
-    </gazebo>
+<robot xmlns:xacro="http://www.ros.org/wiki/xacro">
+  <ros2_control name="RealRobot" type="system">
+    <hardware>
+      <plugin>diffdrive_arduino/DiffDriveArduino</plugin>
+      <param name="left_wheel_name">left_wheel_joint</param>
+      <param name="right_wheel_name">right_wheel_joint</param>
+      <param name="loop_rate">30.0</param>
+      <param name="device">/dev/ttyACM0</param>
+      <param name="baud_rate">57600</param>
+      <param name="timeout">1000</param>
+      <param name="enc_counts_per_rev_left">3450</param>
+      <param name="enc_counts_per_rev_right">3450</param>
+    </hardware>
+    <joint name="left_wheel_joint">
+      <command_interface name="velocity">
+        <param name="min">-10</param>
+        <param name="max">10</param>
+      </command_interface>
+      <state_interface name="position" />
+      <state_interface name="velocity" />
+    </joint>
+    <joint name="right_wheel_joint">
+      <command_interface name="velocity">
+        <param name="min">-10</param>
+        <param name="max">10</param>
+      </command_interface>
+      <state_interface name="position" />
+      <state_interface name="velocity" />
+    </joint>
+  </ros2_control>
 </robot>
